File: optacon/hv_driver.kicad_sch (KiCad schematic)
At the start: 11 parts

Commit message: schematic, footprints
Parts:
- R4: renamed from R(pu); value 3.3k -> (none)
- U3: renamed from U?; value (none) -> DRV2665; footprint (none) -> Package_DFN_QFN:Texas_S-PVQFN-N20_EP2.7x2.7mm_ThermalVias
- renumbered C(vdd) to C1, C(pump) to C2, C(pump) to C3, C(bst) to C4, R(ext) to R3, R(pu) to R5
Changed lines of the file:
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@@
   (symbol (lib_id "power:GND") (at 80.01 81.28 0) (unit 1)
     (in_bom yes) (on_board yes) (fields_autoplaced)
-    (property "Reference" "#PWR?" (id 0) (at 80.01 87.63 0)
-      (effects (font (size 1.27 1.27)) hide)
-    )
-    (property "Value" "" (id 1) (at 80.01 86.36 0))
+    (property "Reference" "#PWR0106" (id 0) (at 80.01 87.63 0)
+      (effects (font (size 1.27 1.27)) hide)
+    )
+    (property "Value" "GND" (id 1) (at 80.01 86.36 0))
     (property "Footprint" "" (id 2) (at 80.01 81.28 0)
       (effects (font (size 1.27 1.27)) hide)
@@
   (symbol (lib_id "Device:C") (at 80.01 77.47 0) (unit 1)
     (in_bom yes) (on_board yes) (fields_autoplaced)
-    (property "Reference" "C(pump)" (id 0) (at 83.82 76.1999 0)
+    (property "Reference" "C2" (id 0) (at 83.82 76.1999 0)
       (effects (font (size 1.27 1.27)) (justify left))
     )
@@
   )
   (symbol (lib_id "power:GND") (at 139.7 83.82 0) (unit 1)
-    (in_bom yes) (on_board yes) (fields_autoplaced)
-    (property "Reference" "#PWR?" (id 0) (at 139.7 90.17 0)
-      (effects (font (size 1.27 1.27)) hide)
-    )
-    (property "Value" "GND" (id 1) (at 139.7 88.9 0))
+    (in_bom yes) (on_board yes)
+    (property "Reference" "#PWR0102" (id 0) (at 139.7 90.17 0)
+      (effects (font (size 1.27 1.27)) hide)
+    )
+    (property "Value" "GND" (id 1) (at 139.7 87.63 0))
     (property "Footprint" "" (id 2) (at 139.7 83.82 0)
       (effects (font (size 1.27 1.27)) hide)
@@
   (symbol (lib_id "Device:C") (at 151.13 68.58 0) (unit 1)
     (in_bom yes) (on_board yes) (fields_autoplaced)
-    (property "Reference" "C(bst)" (id 0) (at 154.94 67.3099 0)
+    (property "Reference" "C4" (id 0) (at 154.94 67.3099 0)
       (effects (font (size 1.27 1.27)) (justify left))
     )
@@
   (symbol (lib_id "power:GND") (at 72.39 106.68 0) (unit 1)
     (in_bom yes) (on_board yes) (fields_autoplaced)
-    (property "Reference" "#PWR?" (id 0) (at 72.39 113.03 0)
-      (effects (font (size 1.27 1.27)) hide)
-    )
-    (property "Value" "" (id 1) (at 72.39 111.76 0))
+    (property "Reference" "#PWR0107" (id 0) (at 72.39 113.03 0)
+      (effects (font (size 1.27 1.27)) hide)
+    )
+    (property "Value" "GND" (id 1) (at 72.39 111.76 0))
     (property "Footprint" "" (id 2) (at 72.39 106.68 0)
       (effects (font (size 1.27 1.27)) hide)
@@
   (symbol (lib_id "power:GND") (at 151.13 72.39 0) (unit 1)
     (in_bom yes) (on_board yes)
-    (property "Reference" "#PWR?" (id 0) (at 151.13 78.74 0)
-      (effects (font (size 1.27 1.27)) hide)
-    )
-    (property "Value" "" (id 1) (at 151.13 76.2 0))
+    (property "Reference" "#PWR0101" (id 0) (at 151.13 78.74 0)
+      (effects (font (size 1.27 1.27)) hide)
+    )
+    (property "Value" "GND" (id 1) (at 151.13 76.2 0))
     (property "Footprint" "" (id 2) (at 151.13 72.39 0)
       (effects (font (size 1.27 1.27)) hide)
@@
   (symbol (lib_id "Device:C") (at 104.14 57.15 0) (unit 1)
     (in_bom yes) (on_board yes) (fields_autoplaced)
-    (property "Reference" "C(vdd)" (id 0) (at 107.95 55.8799 0)
+    (property "Reference" "C1" (id 0) (at 107.95 55.8799 0)
       (effects (font (size 1.27 1.27)) (justify left))
     )
@@
   (symbol (lib_id "Device:C") (at 72.39 102.87 0) (unit 1)
     (in_bom yes) (on_board yes) (fields_autoplaced)
-    (property "Reference" "C(pump)" (id 0) (at 76.2 101.5999 0)
+    (property "Reference" "C3" (id 0) (at 76.2 101.5999 0)
       (effects (font (size 1.27 1.27)) (justify left))
     )
@@
   (symbol (lib_id "Device:R") (at 59.69 88.9 180) (unit 1)
     (in_bom yes) (on_board yes) (fields_autoplaced)
-    (property "Reference" "R(pu)" (id 0) (at 62.23 87.6299 0)
+    (property "Reference" "R5" (id 0) (at 62.23 87.6299 0)
       (effects (font (size 1.27 1.27)) (justify right))
     )
@@
   (symbol (lib_id "Device:R") (at 140.97 91.44 90) (unit 1)
     (in_bom yes) (on_board yes)
-    (property "Reference" "R(ext)" (id 0) (at 140.97 93.98 90))
+    (property "Reference" "R3" (id 0) (at 140.97 93.98 90))
     (property "Value" "" (id 1) (at 140.97 96.52 90))
     (property "Footprint" "" (id 2) (at 140.97 93.218 90)
@@
   )
   (symbol (lib_id "power:GND") (at 119.38 119.38 0) (unit 1)
-    (in_bom yes) (on_board yes) (fields_autoplaced)
-    (property "Reference" "#PWR?" (id 0) (at 119.38 125.73 0)
-      (effects (font (size 1.27 1.27)) hide)
-    )
-    (property "Value" "" (id 1) (at 119.38 124.46 0))
+    (in_bom yes) (on_board yes)
+    (property "Reference" "#PWR0104" (id 0) (at 119.38 125.73 0)
+      (effects (font (size 1.27 1.27)) hide)
+    )
+    (property "Value" "GND" (id 1) (at 119.38 123.19 0))
     (property "Footprint" "" (id 2) (at 119.38 119.38 0)
       (effects (font (size 1.27 1.27)) hide)
@@
   )
   (symbol (lib_id "power:GND") (at 147.32 95.25 0) (unit 1)
-    (in_bom yes) (on_board yes) (fields_autoplaced)
-    (property "Reference" "#PWR?" (id 0) (at 147.32 101.6 0)
-      (effects (font (size 1.27 1.27)) hide)
-    )
-    (property "Value" "" (id 1) (at 147.32 100.33 0))
+    (in_bom yes) (on_board yes)
+    (property "Reference" "#PWR0103" (id 0) (at 147.32 101.6 0)
+      (effects (font (size 1.27 1.27)) hide)
+    )
+    (property "Value" "GND" (id 1) (at 147.32 99.06 0))
     (property "Footprint" "" (id 2) (at 147.32 95.25 0)
       (effects (font (size 1.27 1.27)) hide)
@@
   (symbol (lib_id "Device:R") (at 69.85 88.9 0) (unit 1)
     (in_bom yes) (on_board yes) (fields_autoplaced)
-    (property "Reference" "R(pu)" (id 0) (at 72.39 87.6299 0)
-      (effects (font (size 1.27 1.27)) (justify left))
-    )
-    (property "Value" "3.3k" (id 1) (at 72.39 90.1699 0)
+    (property "Reference" "R4" (id 0) (at 72.39 87.6299 0)
+      (effects (font (size 1.27 1.27)) (justify left))
+    )
+    (property "Value" "" (id 1) (at 72.39 90.1699 0)
       (effects (font (size 1.27 1.27)) (justify left))
     )
@@
   (symbol (lib_id "optacon:DRV2665") (at 119.38 96.52 0) (unit 1)
     (in_bom yes) (on_board yes) (fields_autoplaced)
-    (property "Reference" "U?" (id 0) (at 121.3994 119.38 0)
-      (effects (font (size 1.27 1.27)) (justify left))
-    )
-    (property "Value" "" (id 1) (at 121.3994 121.92 0)
-      (effects (font (size 1.27 1.27)) (justify left))
-    )
-    (property "Footprint" "" (id 2) (at 120.65 118.11 0)
+    (property "Reference" "U3" (id 0) (at 121.3994 119.38 0)
+      (effects (font (size 1.27 1.27)) (justify left))
+    )
+    (property "Value" "DRV2665" (id 1) (at 121.3994 121.92 0)
+      (effects (font (size 1.27 1.27)) (justify left))
+    )
+    (property "Footprint" "Package_DFN_QFN:Texas_S-PVQFN-N20_EP2.7x2.7mm_ThermalVias" (id 2) (at 120.65 118.11 0)
       (effects (font (size 1.27 1.27)) (justify left) hide)
     )
@@
   (symbol (lib_id "power:GND") (at 104.14 60.96 0) (unit 1)
     (in_bom yes) (on_board yes) (fields_autoplaced)
-    (property "Reference" "#PWR?" (id 0) (at 104.14 67.31 0)
-      (effects (font (size 1.27 1.27)) hide)
-    )
-    (property "Value" "" (id 1) (at 104.14 66.04 0))
+    (property "Reference" "#PWR0105" (id 0) (at 104.14 67.31 0)
+      (effects (font (size 1.27 1.27)) hide)
+    )
+    (property "Value" "GND" (id 1) (at 104.14 66.04 0))
     (property "Footprint" "" (id 2) (at 104.14 60.96 0)
       (effects (font (size 1.27 1.27)) hide)
