File: actuator/export/stencil_adhesive/stencil.kicad_pcb (KiCad board)
At the start: 2 copper layers, 94.9 x 105.2 mm, 122 parts, among them J1 Conn_01x12, J2 Conn_01x40_Socket, U1 HV509, U2 HV509, U3 DRV2665

Commit message: rev3.1 gerbers
Parts:
- removed the J2 at (180.1, 73.7)
- removed the J2 at (116.8, 73.7)
- removed the J2 at (148.5, 73.7)
- removed KiKit_FID_B_1, KiKit_FID_B_2, KiKit_FID_B_3, KiKit_FID_T_1, KiKit_FID_T_2, KiKit_FID_T_3: Fiducial, Fiducial
- added J2: Conn_01x40_Socket, Optacon_common:Hirose_FH34SRJ-40S-0.5SH, F.Cu at (116.8, 74.7)
- added J2: Conn_01x40_Socket, Optacon_common:Hirose_FH34SRJ-40S-0.5SH, F.Cu at (180.1, 74.7)
- added J2: Conn_01x40_Socket, Optacon_common:Hirose_FH34SRJ-40S-0.5SH, F.Cu at (148.5, 74.7)
- added REF**: Fiducial, Fiducial, F.Cu at (108.5, 22.5)
- added REF**: Fiducial, Fiducial, F.Cu at (108.5, 122.7)
- added REF**: Fiducial, Fiducial, F.Cu at (188.5, 22.5)
- added REF**: Fiducial, Fiducial, B.Cu at (108.5, 22.5)
- added REF**: Fiducial, Fiducial, B.Cu at (108.5, 122.7)
- added REF**: Fiducial, Fiducial, B.Cu at (188.5, 22.5)
- C8 (x3): value 0.1 -> 0.1 µF
Routing:
- net Board_2-/reed4: track 10.5 -> 12.5 mm
- net Board_0-/reed3: track 10.7 -> 12.7 mm
- net Board_0-/reed2: track 11.0 -> 13.0 mm
- net Board_0-/reed19: track 11.0 -> 13.0 mm
- net Board_0-/reed15: track 9.97 -> 12.0 mm
- net Board_0-/reed1: track 11.6 -> 13.6 mm
- net Board_2-/reed9: track 11.3 -> 13.3 mm
- net Board_2-/reed8: track 10.6 -> 12.6 mm
- net Board_2-/reed7: track 10.0 -> 12.0 mm
- net Board_2-/reed6: track 10.0 -> 12.0 mm
- net Board_2-/reed20: track 11.6 -> 13.6 mm
- net Board_2-/reed2: track 11.0 -> 13.0 mm
- net Board_2-/reed19: track 11.0 -> 13.0 mm
- net Board_2-/reed17: track 10.6 -> 12.6 mm
- net Board_2-/reed16: track 10.4 -> 12.4 mm
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Other:
- board text added: "piezo driver board rev 3.1"
- board text removed: "piezo driver board rev 3"
