File: motherboard/motherboard.kicad_pcb (KiCad board)
At the start: 2 copper layers, 42.9 x 71.7 mm, 49 parts, among them J1 Conn_01x12_MountingPin, J2 Conn_01x12_MountingPin, J3 Conn_01x12_MountingPin, J4 Conn_01x12_MountingPin, J5 Conn_01x12_MountingPin, J6 Conn_01x12_MountingPin, J7 USB_C_Receptacle_USB2.0, SW1 RST, SW2 BOOT, U1 SRV05-4, U2 M3406-ADJ, U3 ESP32-S3-WROOM-1, U4 LM324

Commit message: add/update revision texts
Other:
- board text added: "piezo motherboard rev 2"
Changed lines of the file:
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@@
       ))
   )
+  (gr_rect (start 30.725 91.05) (end 69.575 95.6)
+    (stroke (width 0.15) (type solid)) (fill solid) (layer "B.SilkS"))
   (gr_rect (start 28.9 45.9) (end 71.8 117.55)
     (stroke (width 0.1) (type default)) (fill none) (layer "Edge.Cuts"))
+  (gr_text "piezo motherboard\nrev 2" (at 58.25 89.7) (layer "B.SilkS")
+    (effects (font (size 1 1) (thickness 0.15)) (justify left bottom mirror))
+  )
   (segment (start 36.75 84.13) (end 36.82 84.2) (width 0.3) (layer "F.Cu") (net 1))
   (segment (start 31.93 110.525) (end 30.73 109.325) (width 0.2) (layer "F.Cu") (net 1))
